Commit message: planning robot

File: urdf/modified_robo9_with_planning.urdf (robot description, URDF)
Before this commit: robot robo9, 9 links, 8 joints
Links:
- link base_link: geometry collision mesh filename=package://modified_robo9_with_planning/meshes/base_link.STL; visual mesh filename=package://modified_robo9_with_planning/meshes/base_link.STL
- link base_to_first_link: geometry collision mesh filename=package://modified_robo9_with_planning/meshes/base_to_first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; visual mesh filename=package://modified_robo9_with_planning/meshes/base_to_first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
- link end_effector_link: geometry collision mesh filename=package://modified_robo9_with_planning/meshes/end_effector_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; visual mesh filename=package://modified_robo9_with_planning/meshes/end_effector_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
- link first_link: geometry collision mesh filename=package://modified_robo9_with_planning/meshes/first_link.STL; visual mesh filename=package://modified_robo9_with_planning/meshes/first_link.STL
- link left_wheel: geometry collision mesh filename=package://modified_robo9_with_planning/meshes/left_wheel.STL; visual mesh filename=package://modified_robo9_with_planning/meshes/left_wheel.STL
- link right_wheel: geometry collision mesh filename=package://modified_robo9_with_planning/meshes/right_wheel.S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; visual mesh filename=package://modified_robo9_with_planning/meshes/right_wheel.S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
- link second_link: geometry collision mesh filename=package://modified_robo9_with_planning/meshes/second_link.S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; visual mesh filename=package://modified_robo9_with_planning/meshes/second_link.S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
- link tray_diffusor: geometry collision mesh filename=package://modified_robo9_with_planning/meshes/tray_diffusor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; visual mesh filename=package://modified_robo9_with_planning/meshes/tray_diffusor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

File: urdf/modified_robo9_with_planning.xacro (robot description, xacro)
@@ -1,9 +1,9 @@
 <?xml version="1.0"?>
 <!-- Name your robot here -->
-<robot name ="robo9" xmlns:xacro="http://wiki.ros.org/xacro">
+<robot name ="modified_robo9_with_planning" xmlns:xacro="http://wiki.ros.org/xacro">
 <!-- Include your urdf files here -->
 	<!-- Include Robot's urdf filepath -->
 	<!-- Include Lidar's urdf filepath -->
-	<xacro:include filename="$(find robo9)/urdf/robo9.urdf"/>
+	<xacro:include filename="$(find modified_robo9_with_planning)/urdf/modified_robo9_with_planning.urdf"/>
 	<xacro:macro name="box_inertia" params="mass x y z">
         <inertia ixx="${mass*(y*y+z*z)/12}" ixy = "0" ixz = "0" iyy="${mass*(x*x+z*z)/12}" iyz = "0" izz="${mass*(x*x+y*y)/12}" />
@@ -32,5 +32,5 @@
 		<!-- <topic>__default_topic__</topic>/ -->
 		<plugin filename="libgazebo_ros_imu_sensor.so" name="imu_plugin">
-			<topicName>/robo9/imu</topicName>
+			<topicName>/modified_robo9_with_planning/imu</topicName>
 			<bodyName>imu_link</bodyName>
 			<updateRateHZ>10.0</updateRateHZ>
@@ -47,5 +47,5 @@
 	<gazebo>
 		<plugin name="gazebo_ros_control" filename="libgazebo_ros_control.so">
-			<robotNamespace>/robo9</robotNamespace>
+			<robotNamespace>/modified_robo9_with_planning</robotNamespace>
 			<robotSimType>gazebo_ros_control/DefaultRobotHWSim</robotSimType>
 			<legacyModeNS>true</legacyModeNS>
@@ -65,5 +65,5 @@
 			<alwaysOn>true</alwaysOn>
 			<legacyMode>false</legacyMode>
-			<updateRate>20</updateRate>
+			<updateRate>30</updateRate>
 			<leftJoint>left_wheel_joint</leftJoint>
 			<rightJoint>right_wheel_joint</rightJoint>
@@ -73,7 +73,7 @@
 			<!-- 8 in to m-> 0.2032 -->
 			<wheelTorque>40</wheelTorque>
-			<wheelAcceleration>1.0</wheelAcceleration>
-			<commandTopic>/robo9/cmd_vel</commandTopic>
-			<odometryTopic>/robo9/odom</odometryTopic>
+			<wheelAcceleration>5.0</wheelAcceleration>
+			<commandTopic>/modified_robo9_with_planning/cmd_vel</commandTopic>
+			<odometryTopic>/modified_robo9_with_planning/odom</odometryTopic>
 			<odometryFrame>odom</odometryFrame>
 			<robotBaseFrame>dummy_link</robotBaseFrame>
